File: PCB/ATmega328P-board/ATmega328P-board.kicad_pcb (KiCad board)
At the start: 2 copper layers, 87.4 x 57.8 mm, 28 parts, among them J1 Jack-DC, J2 Headers, J3 Headers, J4 Headers, J5 Headers, J6 Conn_02x03_Odd_Even, J7 Power Screw Terminal, SW1 SW_Push, U1 ATmega328-P, U3 AMS1117, U4 AMS1117, Y1 16MHz

Commit message: Work
Parts:
- removed J2, J3, J4, J5: Headers, Connector_PinHeader_2.54mm:PinHeader_1x06_P2.54mm_Vertical
- added J10: PWM Header, Connector_PinHeader_2.54mm:PinHeader_1x04_P2.54mm_Vertical, F.Cu at (126.5, 144.0)
- added J11: PWM Header, Connector_PinHeader_2.54mm:PinHeader_1x04_P2.54mm_Vertical, F.Cu at (139.6, 98.5)
- added J12: PWM Header, Connector_PinHeader_2.54mm:PinHeader_1x04_P2.54mm_Vertical, F.Cu at (122.8, 106.7)
- added J8: PWM Header, Connector_PinHeader_2.54mm:PinHeader_1x04_P2.54mm_Vertical, F.Cu at (122.8, 119.7)
- added J9: Header, Connector_PinHeader_2.54mm:PinHeader_1x04_P2.54mm_Vertical, F.Cu at (122.8, 131.2)
- C1: footprint Capacitor_THT:CP_Radial_D5.0mm_P2.00mm -> Capacitor_THT:CP_Radial_D5.0mm_P2.50mm
- C3, C4, C6, C7, C8, C9: footprint Capacitor_THT:C_Disc_D5.0mm_W2.5mm_P5.00mm -> Capacitor_SMD:C_0805_2012Metric
- J7: footprint Connector_Phoenix_SPT:PhoenixContact_SPT_1.5_3-H-3.5_1x03_P3.5mm_Horizontal -> TerminalBlock_Altech:Altech_AK100_1x03_P5.00mm
- R1, R2, R3: footprint Resistor_THT:R_Axial_DIN0204_L3.6mm_D1.6mm_P7.62mm_Horizontal -> Resistor_SMD:R_0805_2012Metric
- moved J7 9.04 mm to (124.8, 98.9), turned to 0 degrees
- moved C3 6.07 mm to (134.8, 124.0)
- moved R2 3.64 mm to (171.2, 112.8)
- moved D2 2.80 mm to (166.0, 117.0)
- moved C6 2.37 mm to (164.0, 112.5)
- moved C7 1.80 mm to (161.1, 127.0)
- moved C4 1.07 mm to (134.8, 132.2)
- moved R1 0.81 mm to (144.2, 112.0), turned to -90 degrees
Routing:
- net VCC: track 160.0 -> 225.2 mm, vias 2 -> 4
- net /+3.3: track 92.7 -> 144.0 mm, vias 4 -> 2
- net /TX: track 10.2 -> 42.9 mm, vias 0 -> 5
- net /PD5: track 14.4 -> 44.6 mm, vias 0 -> 2
- net /RX: track 13.1 -> 42.7 mm, vias 0 -> 2
- net /DTR: track 12.7 -> 39.0 mm, vias 0 -> 2
- net /PC3: track 39.9 -> 17.6 mm, vias 2 -> 1
- net /PC2: track 42.4 -> 21.7 mm, vias 2 -> 1
- net /PD2: track 33.0 -> 51.1 mm, vias 2 -> 4
- net /PB0: track 25.8 -> 43.7 mm
- net /PC1: track 41.7 -> 27.2 mm, vias 2 -> 1
- net /PB1: track 34.0 -> 44.9 mm, vias 2 -> 0
- net /PB2: track 34.4 -> 44.6 mm
- net /PD4: track 27.2 -> 37.2 mm
- net /SCK: track 45.5 -> 51.9 mm
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Other:
- outline, holes or cut-outs redrawn
- board text added: "+3.3V"
- board text added: "DTR"
- board text added: "GND"
- board text added: "MISO"
- board text added: "MOSI"
- board text added: "PB0"
- board text added: "PB1"
- board text added: "PB2"
- board text added: "PC0"
- board text added: "PC1"
- board text added: "PC2"
- board text added: "PC3"
- board text added: "PC4"
- board text added: "PC5"
- board text added: "PD3"
- board text added: "PD5"
- board text added: "PWM"
- board text added: "RESET"
- board text added: "RX"
- board text added: "SCK"
- board text added: "TX"
- board text added: "VCC"
