File: PCB/ATmega328P-board/ATmega328P-board.kicad_sch (KiCad schematic)
At the start: 24 parts, among them J1 Jack-DC, J2 Headers, J3 Headers, J4 Headers, J5 Headers, J6 Conn_02x03_Odd_Even, SW1 SW_Push, U1 ATmega328-P, U3 AMS1117, U4 AMS1117, Y1 16MHz

Commit message: 2hwork
Parts:
- removed C5: 100nF, Capacitor_THT:C_Disc_D5.0mm_W2.5mm_P5.00mm, symbol Device:C
- added D2, D3: LED, LED_THT:LED_D3.0mm, symbol Device:LED
- added J7: Power Screw Terminal, Connector_Phoenix_SPT:PhoenixContact_SPT_1.5_3-H-3.5_1x03_P3.5mm_Horizontal, symbol Connector:Screw_Terminal_01x03
- added R2, R3: 1K, Resistor_THT:R_Axial_DIN0204_L3.6mm_D1.6mm_P7.62mm_Horizontal, symbol Device:R
- C1, C10: footprint Capacitor_THT:C_Rect_L7.2mm_W2.5mm_P5.00mm -> Capacitor_THT:CP_Radial_D5.0mm_P2.00mm
- R1: footprint Diode_THT:D_DO-41_SOD81_P10.16mm_Horizontal -> Resistor_THT:R_Axial_DIN0204_L3.6mm_D1.6mm_P7.62mm_Horizontal
Connections:
- net +3.3: now also J7.2 (Pin_2)
- net GND: now also J6.6 (Pin_6), D2.2 (A), D3.2 (A), J7.3 (Pin_3)
- net PB1: no longer J2.3 (Pin_3), J2.4 (Pin_4), U1.16 (PB2)
- net SCK: now also R3.2
- net VCC: now also J6.2 (Pin_2), U1.21 (AREF), J7.1 (Pin_1), R2.2
- net RESET: now reaches C9.2, R1.1, SW1.1, U1.1 (~{RESET}/PC6)
- net RESET: now also J6.5 (Pin_5)
- new net: D3.1 (K), R3.1
- new net: D2.1 (K), R2.1
- new net PB2: J2.4 (Pin_4), U1.16 (PB2)
Other:
- title: (none) -> ATmega328P Custom Board

Commit message: Work
Parts:
- removed J2, J3, J4, J5: Headers, Connector_PinHeader_2.54mm:PinHeader_1x06_P2.54mm_Vertical, symbol Connector:Conn_01x06_Pin
- added J10, J11, J12, J8: PWM Header, Connector_PinHeader_2.54mm:PinHeader_1x04_P2.54mm_Vertical, symbol Connector:Conn_01x04_Pin
- added J9: Header, Connector_PinHeader_2.54mm:PinHeader_1x04_P2.54mm_Vertical, symbol Connector:Conn_01x04_Pin
- C1: footprint Capacitor_THT:CP_Radial_D5.0mm_P2.00mm -> Capacitor_THT:CP_Radial_D5.0mm_P2.50mm
- C3, C4, C6, C7, C8, C9: footprint Capacitor_THT:C_Disc_D5.0mm_W2.5mm_P5.00mm -> Capacitor_SMD:C_0805_2012Metric
- J7: footprint Connector_Phoenix_SPT:PhoenixContact_SPT_1.5_3-H-3.5_1x03_P3.5mm_Horizontal -> TerminalBlock_Altech:Altech_AK100_1x03_P5.00mm
- R1, R2, R3: footprint Resistor_THT:R_Axial_DIN0204_L3.6mm_D1.6mm_P7.62mm_Horizontal -> Resistor_SMD:R_0805_2012Metric
Connections:
- net +3.3: now also J10.1 (Pin_1)
- net DTR: now also J9.3 (Pin_3)
- net GND: now also J12.4 (Pin_4), J9.4 (Pin_4)
- net PB0: now also J12.3 (Pin_3)
- net PB1: now also J8.2 (Pin_2)
- net PB2: now also J8.1 (Pin_1)
- net PC0: now also J11.1 (Pin_1)
- net PC1: now also J11.2 (Pin_2)
- net PC2: now also J11.3 (Pin_3)
- net PC3: now also J11.4 (Pin_4)
- net PC4: now also J12.1 (Pin_1)
- net PC5: now also J12.2 (Pin_2)
- net PD2: now also J10.3 (Pin_3)
- net PD3: now also J8.3 (Pin_3)
- net PD4: now also J10.4 (Pin_4)
- net PD5: now also J8.4 (Pin_4)
- net RX: now also J9.2 (Pin_2)
- net TX: now also J9.1 (Pin_1)
- net VCC: now also J10.2 (Pin_2)
- no-connect marks 9 -> 4

Commit message: another work
Parts:
- J10, J11, J12: value PWM Header -> Header
Changed lines of the file:
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@@
 			)
 		)
-		(property "Value" "PWM Header"
+		(property "Value" "Header"
 			(at 262.636 89.154 0)
 			(show_name no)
@@
 			)
 		)
-		(property "Value" "PWM Header"
+		(property "Value" "Header"
 			(at 262.636 61.214 0)
 			(show_name no)
@@
 			)
 		)
-		(property "Value" "PWM Header"
+		(property "Value" "Header"
 			(at 262.636 75.184 0)
 			(show_name no)
